File: Schematic/Pixsso/Pixsso.kicad_sch (KiCad schematic)
At the start: 9 parts

Commit message: Schematic update
Connections:
- new net Display_PWR: M1. (gnd), U1. (VCC)
Changed lines of the file:
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@@
-	)
-	(junction
-		(at 39.37 118.11)
-		(diameter 0)
-		(color 0 0 0 0)
 	)
 	(junction
@@
 	(wire
 		(pts
-			(xy 39.37 120.65) (xy 39.37 118.11)
-		)
-		(stroke
-			(width 0)
-			(type default)
-		)
-	)
-	(wire
-		(pts
 			(xy 68.58 158.75) (xy 63.5 158.75)
 		)
@@
 	(wire
 		(pts
-			(xy 39.37 115.57) (xy 39.37 118.11)
+			(xy 39.37 115.57) (xy 39.37 120.65)
 		)
 		(stroke
@@
 	(wire
 		(pts
+			(xy 109.22 163.83) (xy 106.68 163.83)
+		)
+		(stroke
+			(width 0)
+			(type default)
+		)
+	)
+	(wire
+		(pts
 			(xy 54.61 125.73) (xy 68.58 125.73)
 		)
@@
 		(pts
 			(xy 106.68 130.81) (xy 118.11 130.81)
-		)
-		(stroke
-			(width 0)
-			(type default)
-		)
-	)
-	(wire
-		(pts
-			(xy 35.56 118.11) (xy 39.37 118.11)
 		)
 		(stroke
@@
 	(global_label "Display_CS"
 		(shape input)
-		(at 35.56 118.11 180)
+		(at 109.22 163.83 0)
 		(fields_autoplaced yes)
 		(effects
@@
 				(size 1.27 1.27)
 			)
-			(justify right)
+			(justify left)
 		)
 		(property "Intersheetrefs" "${INTERSHEET_REFS}"
-			(at 22.294 118.11 0)
+			(at 122.486 163.83 0)
 			(effects
 				(font
 					(size 1.27 1.27)
 				)
-				(justify right)
+				(justify left)
 				(hide yes)
 			)
